File: KiCad/T-Wall/T-Wall.kicad_sch (KiCad schematic)
At the start: 9 parts, among them U1 TCA9555DBR

Commit message: EOD 11.03
Parts:
- removed A1: RaspberryPi_Pico, Module:RaspberryPi_Pico_SMD, symbol MCU_Module:RaspberryPi_Pico_Extensive
- removed R3: 10k, symbol Device:R
- added C2, C3, C4: 100n, Capacitor_SMD:C_0402_1005Metric, symbol Device:C
- added JP10, JP4, JP7: JP_A1, Jumper:SolderJumper-3_P1.3mm_Open_RoundedPad1.0x1.5mm, symbol Jumper:SolderJumper_3_Open
- added JP11, JP5, JP8: JP_A2, Jumper:SolderJumper-3_P1.3mm_Open_RoundedPad1.0x1.5mm, symbol Jumper:SolderJumper_3_Open
- added JP3, JP6, JP9: JP_A0, Jumper:SolderJumper-3_P1.3mm_Open_RoundedPad1.0x1.5mm, symbol Jumper:SolderJumper_3_Open
- added U2: SN74AHCT125N, SN74AHCT125N:DIP794W45P254L1930H508Q14, symbol SN74AHCT125N:SN74AHCT125N
- added U3: ESP32-S3-DevKitC, PCM_Espressif:ESP32-S3-DevKitC, symbol Espressif:ESP32-S3-DevKitC
- added U4, U5, U6: TCA9555DBR, Package_SO:SSOP-24_5.3x8.2mm_P0.65mm, symbol Interface_Expansion:TCA9555DBR
- C1: footprint (none) -> Capacitor_SMD:C_0402_1005Metric
- JP0, JP1, JP2: footprint (none) -> Jumper:SolderJumper-3_P1.3mm_Open_RoundedPad1.0x1.5mm
- R1, R2: footprint (none) -> Resistor_SMD:R_0402_1005Metric
Connections:
- net GND: now also JP0.3 (B), JP1.3 (B), JP2.3 (B), C2.2, C3.2, C4.2, JP10.3 (B), JP11.3 (B), JP3.3 (B), JP4.3 (B), JP5.3 (B), JP6.3 (B), JP7.3 (B), JP8.3 (B), JP9.3 (B), U2.1 (1~{OE}), U2.10 (3~{OE}), U2.12 (4A), U2.13 (4~{OE}), U2.4 (2~{OE}), U2.5 (2A), U2.7 (GND), U2.9 (3A), U3.22 (GND), U3.23 (GND), U3.24 (GND), U3.44 (GND), U4.12 (GND), U5.12 (GND), U6.12 (GND); no longer JP0.1 (A), JP1.1 (A), JP2.1 (A)
- net I2C_SCL: now also R2.2, U3.15 (GPIO9/ADC1_CH8), U4.22 (SCL), U5.22 (SCL), U6.22 (SCL); no longer R2.1
- net I2C_SDA: now also R1.1, U3.12 (GPIO8/ADC1_CH7), U4.23 (SDA), U5.23 (SDA), U6.23 (SDA); no longer R1.2
- net INT_000: now reaches U1.1 (~{INT})
- net INT_000: now also U3.4 (GPIO4/ADC1_CH3)
- removed net VCC_3.3: C1.1, JP0.3 (B), JP1.3 (B), JP2.3 (B), R1.1, R2.2, U1.24 (VCC)
- new net: JP10.2 (C), U6.2 (A1)
- new net: JP9.2 (C), U6.21 (A0)
- new net: JP11.2 (C), U6.3 (A2)
- new net: JP4.2 (C), U4.2 (A1)
- new net: JP3.2 (C), U4.21 (A0)
- new net: JP5.2 (C), U4.3 (A2)
- new net: JP8.2 (C), U5.3 (A2)
- new net: JP7.2 (C), U5.2 (A1)
- new net: JP6.2 (C), U5.21 (A0)
- new net +3.3V: C1.1, C2.1, C3.1, C4.1, JP0.1 (A), JP1.1 (A), JP10.1 (A), JP11.1 (A), JP2.1 (A), JP3.1 (A), JP4.1 (A), JP5.1 (A), JP6.1 (A), JP7.1 (A), JP8.1 (A), JP9.1 (A), R1.2, R2.1, U1.24 (VCC), U3.1 (3V3), U3.2 (3V3), U4.24 (VCC), U5.24 (VCC), U6.24 (VCC)
- new net +5V: U2.14 (VCC), U3.21 (5V)
- new net INT_001: U3.5 (GPIO5/ADC1_CH4), U4.1 (~{INT})
- new net INT_010: U3.6 (GPIO6/ADC1_CH5), U5.1 (~{INT})
- new net INT_011: U3.7 (GPIO7/ADC1_CH6), U6.1 (~{INT})
- new net LEDS: U2.2 (1A), U3.41 (GPIO1/ADC1_CH0)
- no-connect marks 0 -> 34
Other:
- moved on the sheet: R1, R2
