File: KiCad/T-Wall/_autosave-T-Wall.kicad_pcb (KiCad board)
At the start: 2 copper layers, 137 x 65 mm, 34 parts, among them J1 Conn_1, J2 Conn_2, J3 Conn_3, J4 Conn_4, J5 Conn_5, J6 Conn_6, J7 Conn_7, J8 Conn_8, J9 2086-1203_700-000_997-605, U1 TCA9555DBR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

Commit message: PCB Revision 1
Routing:
- net /Sensor_R5S8: track 24.7 -> 29.8 mm
- net /Sensor_R5S7: track 25.8 -> 27.3 mm
- net /Sensor_R5S1: track 35.8 -> 36.8 mm
- net /Sensor_R8S1: track 82.2 -> 83.2 mm
- net /Sensor_R5S2: track 37.5 -> 38.5 mm
- net /Sensor_R5S5: track 29.5 -> 30.4 mm
- net /Sensor_R5S3: track 32.7 -> 33.6 mm
- net /Sensor_R5S6: track 31.3 -> 32.1 mm
- net /Sensor_R5S4: track 34.4 -> 35.3 mm
