File: KiCad/T-Wall/_autosave-T-Wall.kicad_sch (KiCad schematic)
At the start: 25 parts, among them J1 2086-1203_700-000_997-605, U1 TCA9555DBR, U2 SN74AHCT125N, U3 ESP32-S3-DevKitC, U4 TCA9555DBR, U5 TCA9555DBR, U6 TCA9555DBR

Commit message: PCB Revision 1
Parts:
- added J1: Conn_1, Connector_IDC:IDC-Header_2x05_P2.54mm_Vertical, symbol Connector_Generic:Conn_01x10
- added J2: Conn_2, Connector_IDC:IDC-Header_2x05_P2.54mm_Vertical, symbol Connector_Generic:Conn_01x10
- added J3: Conn_3, Connector_IDC:IDC-Header_2x05_P2.54mm_Vertical, symbol Connector_Generic:Conn_01x10
- added J4: Conn_4, Connector_IDC:IDC-Header_2x05_P2.54mm_Vertical, symbol Connector_Generic:Conn_01x10
- added J5: Conn_5, Connector_IDC:IDC-Header_2x05_P2.54mm_Vertical, symbol Connector_Generic:Conn_01x10
- added J6: Conn_6, Connector_IDC:IDC-Header_2x05_P2.54mm_Vertical, symbol Connector_Generic:Conn_01x10
- added J7: Conn_7, Connector_IDC:IDC-Header_2x05_P2.54mm_Vertical, symbol Connector_Generic:Conn_01x10
- added J8: Conn_8, Connector_IDC:IDC-Header_2x05_P2.54mm_Vertical, symbol Connector_Generic:Conn_01x10
- added R3: 330, Resistor_SMD:R_0402_1005Metric, symbol Device:R
- U2, U3: now not fitted
- renumbered J1 to J9
Connections:
- net +3.3V: now also J1.9 (Pin_9), J2.9 (Pin_9), J3.9 (Pin_9), J4.9 (Pin_9), J5.9 (Pin_9), J6.9 (Pin_9), J7.9 (Pin_9), J8.9 (Pin_9)
- net GND: now also J1.10 (Pin_10), J2.10 (Pin_10), J3.10 (Pin_10), J4.10 (Pin_10), J5.10 (Pin_10), J6.10 (Pin_10), J7.10 (Pin_10), J8.10 (Pin_10)
- net LEDS_OUT: now also R3.1; no longer U2.3 (1Y)
- net Sensor_R7S7: now reaches U6.10 (P06)
- net Sensor_R7S7: now also J7.7 (Pin_7)
- net Sensor_R7S8: now reaches U6.11 (P07)
- net Sensor_R7S8: now also J7.8 (Pin_8)
- net Sensor_R8S1: now reaches U6.13 (P10)
- net Sensor_R8S1: now also J8.1 (Pin_1)
- net Sensor_R8S2: now reaches U6.14 (P11)
- net Sensor_R8S2: now also J8.2 (Pin_2)
- net Sensor_R8S3: now reaches U6.15 (P12)
- net Sensor_R8S3: now also J8.3 (Pin_3)
- net Sensor_R8S4: now reaches U6.16 (P13)
- net Sensor_R8S4: now also J8.4 (Pin_4)
- net Sensor_R8S5: now reaches U6.17 (P14)
- net Sensor_R8S5: now also J8.5 (Pin_5)
- net Sensor_R8S6: now reaches U6.18 (P15)
- net Sensor_R8S6: now also J8.6 (Pin_6)
- net Sensor_R8S7: now reaches U6.19 (P16)
- net Sensor_R8S7: now also J8.7 (Pin_7)
- net Sensor_R8S8: now reaches U6.20 (P17)
- net Sensor_R8S8: now also J8.8 (Pin_8)
- net Sensor_R7S1: now reaches U6.4 (P00)
- net Sensor_R7S1: now also J7.1 (Pin_1)
- net Sensor_R7S2: now reaches U6.5 (P01)
- net Sensor_R7S2: now also J7.2 (Pin_2)
- net Sensor_R7S3: now reaches U6.6 (P02)
- net Sensor_R7S3: now also J7.3 (Pin_3)
- net Sensor_R7S4: now reaches U6.7 (P03)
- net Sensor_R7S4: now also J7.4 (Pin_4)
- net Sensor_R7S5: now reaches U6.8 (P04)
- net Sensor_R7S5: now also J7.5 (Pin_5)
- net Sensor_R7S6: now reaches U6.9 (P05)
- net Sensor_R7S6: now also J7.6 (Pin_6)
- net Sensor_R3S7: now reaches U4.10 (P06)
- net Sensor_R3S7: now also J3.7 (Pin_7)
- net Sensor_R3S8: now reaches U4.11 (P07)
- net Sensor_R3S8: now also J3.8 (Pin_8)
- net Sensor_R4S1: now reaches U4.13 (P10)
- net Sensor_R4S1: now also J4.1 (Pin_1)
- net Sensor_R4S2: now reaches U4.14 (P11)
- net Sensor_R4S2: now also J4.2 (Pin_2)
- net Sensor_R4S3: now reaches U4.15 (P12)
- net Sensor_R4S3: now also J4.3 (Pin_3)
- net Sensor_R4S4: now reaches U4.16 (P13)
- net Sensor_R4S4: now also J4.4 (Pin_4)
- net Sensor_R4S5: now reaches U4.17 (P14)
- net Sensor_R4S5: now also J4.5 (Pin_5)
- net Sensor_R4S6: now reaches U4.18 (P15)
- net Sensor_R4S6: now also J4.6 (Pin_6)
- net Sensor_R4S7: now reaches U4.19 (P16)
- net Sensor_R4S7: now also J4.7 (Pin_7)
- net Sensor_R4S8: now reaches U4.20 (P17)
- net Sensor_R4S8: now also J4.8 (Pin_8)
- net Sensor_R3S1: now reaches U4.4 (P00)
- net Sensor_R3S1: now also J3.1 (Pin_1)
- net Sensor_R3S2: now reaches U4.5 (P01)
- net Sensor_R3S2: now also J3.2 (Pin_2)
- net Sensor_R3S3: now reaches U4.6 (P02)
- net Sensor_R3S3: now also J3.3 (Pin_3)
- net Sensor_R3S4: now reaches U4.7 (P03)
- net Sensor_R3S4: now also J3.4 (Pin_4)
- net Sensor_R3S5: now reaches U4.8 (P04)
- net Sensor_R3S5: now also J3.5 (Pin_5)
- net Sensor_R3S6: now reaches U4.9 (P05)
- net Sensor_R3S6: now also J3.6 (Pin_6)
- net Sensor_R5S7: now reaches U5.10 (P06)
- net Sensor_R5S7: now also J5.7 (Pin_7)
- net Sensor_R5S8: now reaches U5.11 (P07)
- net Sensor_R5S8: now also J5.8 (Pin_8)
- net Sensor_R6S1: now reaches U5.13 (P10)
- net Sensor_R6S1: now also J6.1 (Pin_1)
- net Sensor_R6S2: now reaches U5.14 (P11)
- net Sensor_R6S2: now also J6.2 (Pin_2)
- net Sensor_R6S3: now reaches U5.15 (P12)
- net Sensor_R6S3: now also J6.3 (Pin_3)
- net Sensor_R6S4: now reaches U5.16 (P13)
- net Sensor_R6S4: now also J6.4 (Pin_4)
- net Sensor_R6S5: now reaches U5.17 (P14)
- net Sensor_R6S5: now also J6.5 (Pin_5)
- net Sensor_R6S6: now reaches U5.18 (P15)
- net Sensor_R6S6: now also J6.6 (Pin_6)
- net Sensor_R6S7: now reaches U5.19 (P16)
- net Sensor_R6S7: now also J6.7 (Pin_7)
- net Sensor_R6S8: now reaches U5.20 (P17)
- net Sensor_R6S8: now also J6.8 (Pin_8)
- net Sensor_R5S1: now reaches U5.4 (P00)
- net Sensor_R5S1: now also J5.1 (Pin_1)
- net Sensor_R5S2: now reaches U5.5 (P01)
- net Sensor_R5S2: now also J5.2 (Pin_2)
- net Sensor_R5S3: now reaches U5.6 (P02)
- net Sensor_R5S3: now also J5.3 (Pin_3)
- net Sensor_R5S4: now reaches U5.7 (P03)
- net Sensor_R5S4: now also J5.4 (Pin_4)
- net Sensor_R5S5: now reaches U5.8 (P04)
- net Sensor_R5S5: now also J5.5 (Pin_5)
- net Sensor_R5S6: now reaches U5.9 (P05)
- net Sensor_R5S6: now also J5.6 (Pin_6)
- net Sensor_R1S7: now reaches U1.10 (P06)
- net Sensor_R1S7: now also J1.7 (Pin_7)
- net Sensor_R1S8: now reaches U1.11 (P07)
- net Sensor_R1S8: now also J1.8 (Pin_8)
- net Sensor_R2S1: now reaches U1.13 (P10)
- net Sensor_R2S1: now also J2.1 (Pin_1)
- net Sensor_R2S2: now reaches U1.14 (P11)
- net Sensor_R2S2: now also J2.2 (Pin_2)
- net Sensor_R2S3: now reaches U1.15 (P12)
- net Sensor_R2S3: now also J2.3 (Pin_3)
- net Sensor_R2S4: now reaches U1.16 (P13)
- net Sensor_R2S4: now also J2.4 (Pin_4)
- net Sensor_R2S5: now reaches U1.17 (P14)
- net Sensor_R2S5: now also J2.5 (Pin_5)
- net Sensor_R2S6: now reaches U1.18 (P15)
- net Sensor_R2S6: now also J2.6 (Pin_6)
- net Sensor_R2S7: now reaches U1.19 (P16)
- net Sensor_R2S7: now also J2.7 (Pin_7)
- net Sensor_R2S8: now reaches U1.20 (P17)
- net Sensor_R2S8: now also J2.8 (Pin_8)
- net Sensor_R1S1: now reaches U1.4 (P00)
- net Sensor_R1S1: now also J1.1 (Pin_1)
- net Sensor_R1S2: now reaches U1.5 (P01)
- net Sensor_R1S2: now also J1.2 (Pin_2)
- net Sensor_R1S3: now reaches U1.6 (P02)
- net Sensor_R1S3: now also J1.3 (Pin_3)
- net Sensor_R1S4: now reaches U1.7 (P03)
- net Sensor_R1S4: now also J1.4 (Pin_4)
- net Sensor_R1S5: now reaches U1.8 (P04)
- net Sensor_R1S5: now also J1.5 (Pin_5)
- net Sensor_R1S6: now reaches U1.9 (P05)
- net Sensor_R1S6: now also J1.6 (Pin_6)
- new net: R3.2, U2.3 (1Y)
Other:
- moved on the sheet: C1, C2, C3, C4, J9, JP0, JP1, JP10, JP11, JP2, JP3, JP4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
