File: KiCad/T-Wall/T-Wall.kicad_pcb (KiCad board)
At the start: 2 copper layers, 137 x 65 mm, 34 parts, among them J1 Conn_1, J2 Conn_2, J3 Conn_3, J4 Conn_4, J5 Conn_5, J6 Conn_6, J7 Conn_7, J8 Conn_8, J9 2086-1203_700-000_997-605, U1 TCA9555DBR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

Commit message: PCB Revision 2
Parts:
- added R4: 4.7k, Resistor_SMD:R_0402_1005Metric, F.Cu at (111.0, 53.5)
- added R5: 4.7k, Resistor_SMD:R_0402_1005Metric, F.Cu at (111.0, 51.5)
- added R6: 4.7k, Resistor_SMD:R_0402_1005Metric, F.Cu at (114.5, 112.5)
- added R7: 4.7k, Resistor_SMD:R_0402_1005Metric, F.Cu at (114.5, 108.5)
- moved R3 9.15 mm to (147.0, 88.5)
Routing:
- net +3.3V: track 300.2 -> 323.4 mm, vias 2 -> 4
- net /LEDS_OUT: track 33.7 -> 22.9 mm, vias 2 -> 0
- net Net-(U2-1Y): track 1.55 -> 9.95 mm
- net /Sensor_R5S8: track 24.7 -> 29.8 mm
- net /INT_010: track 82.1 -> 83.7 mm
- net /INT_011: track 62.3 -> 63.8 mm
- net /Sensor_R5S7: track 25.8 -> 27.3 mm
- net /Sensor_R5S1: track 35.8 -> 36.8 mm
- net /Sensor_R5S4: track 34.4 -> 35.4 mm
- net /Sensor_R8S1: track 82.2 -> 83.2 mm
- net /Sensor_R5S2: track 37.5 -> 38.5 mm
- net /INT_001: track 35.3 -> 36.2 mm
- net /Sensor_R5S5: track 29.5 -> 30.4 mm
- net /Sensor_R5S3: track 32.7 -> 33.6 mm
- net /Sensor_R5S6: track 31.3 -> 32.1 mm
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
Commit message: EOD 1303
Parts:
- added C5: 10u, Capacitor_SMD:C_1206_3216Metric_Pad1.33x1.80mm_HandSolder, F.Cu at (150.0, 52.0)
- added C6: 10u, Capacitor_SMD:C_1206_3216Metric_Pad1.33x1.80mm_HandSolder, F.Cu at (160.0, 53.5)
- added R10: 330, Resistor_SMD:R_0402_1005Metric_Pad0.72x0.64mm_HandSolder, F.Cu at (149.5, 88.5)
- added R11: 330, Resistor_SMD:R_0402_1005Metric_Pad0.72x0.64mm_HandSolder, F.Cu at (152.0, 88.5)
- added R12: 330, Resistor_SMD:R_0402_1005Metric_Pad0.72x0.64mm_HandSolder, F.Cu at (154.5, 88.6)
- added R8: 10k, Resistor_SMD:R_0402_1005Metric_Pad0.72x0.64mm_HandSolder, F.Cu at (155.5, 55.5)
- added R9: 10k, Resistor_SMD:R_0402_1005Metric_Pad0.72x0.64mm_HandSolder, F.Cu at (154.0, 55.5)
- added U7: LMZM23601V3, Package_LGA:Texas_SIL0010A_MicroSiP-10-1EP_3.8x3mm_P0.6mm_EP0.7x2.9mm_ThermalVias, F.Cu at (155.7, 52.5)
- C1, C2, C3, C4: footprint Capacitor_SMD:C_0402_1005Metric -> Capacitor_SMD:C_0402_1005Metric_Pad0.74x0.62mm_HandSolder
- J9: value 2086-1203_700-000_997-605 -> 2086-1208/700-000/997-607; footprint 2086-1203_700-000_997-605:WAGO_2086-1203_700-000_997-605 -> 2086-1208_700-000_997-607:2086-1208_700-000_997-607
- R1, R2, R3: footprint Resistor_SMD:R_0402_1005Metric -> Resistor_SMD:R_0402_1005Metric_Pad0.72x0.64mm_HandSolder
- R4, R5, R6, R7: value 4.7k -> 10k; footprint Resistor_SMD:R_0402_1005Metric -> Resistor_SMD:R_0402_1005Metric_Pad0.72x0.64mm_HandSolder
- moved J9 8.63 mm to (152.1, 72.2)
- moved R4 0.10 mm to (111.1, 53.6)
- turned R3 to -90 degrees
- renumbered U4 to U2, U5 to U3, U6 to U4, U3 to U5, U2 to U6
Connections:
- net /LEDS_OUT renamed /LEDS_OUT_1
- U5 pad 1: +3.3V -> unconnected-(U5-3V3-Pad1)_1
- U5 pad 16: unconnected-(U3-GPIO10/ADC1_CH9-Pad16) -> /LEDS_GPIO_1
- U5 pad 17: unconnected-(U3-GPIO11/ADC2_CH0-Pad17) -> /LEDS_GPIO_2
- U5 pad 18: unconnected-(U3-GPIO12/ADC2_CH1-Pad18) -> /LEDS_GPIO_4
- U5 pad 19: unconnected-(U3-GPIO13/ADC2_CH2-Pad19) -> /LEDS_GPIO_3
- U5 pad 2: +3.3V -> unconnected-(U5-3V3-Pad1)
- U5 pad 28: unconnected-(U3-GPIO47-Pad28) -> /LEDS_DATA_EN
- U5 pad 29: unconnected-(U3-GPIO48-Pad29) -> /LEDS_PWR_EN
- U5 pad 40: unconnected-(U3-GPIO2/ADC1_CH1-Pad40) -> /DCDC_PGood
- U5 pad 41: /LEDS_GPIO -> /DCDC_EN
- U6 pad 1: GND -> /LEDS_DATA_EN
- U6 pad 10: GND -> /LEDS_DATA_EN
- U6 pad 11: unconnected-(U2-4Y-Pad11) -> Net-(U6-4Y)
- U6 pad 12: GND -> /LEDS_GPIO_4
- U6 pad 13: GND -> /LEDS_DATA_EN
- U6 pad 2: /LEDS_GPIO -> /LEDS_GPIO_1
- U6 pad 4: GND -> /LEDS_DATA_EN
- U6 pad 5: GND -> /LEDS_GPIO_2
- U6 pad 6: unconnected-(U2-2Y-Pad6) -> Net-(U6-2Y)
- U6 pad 8: unconnected-(U2-3Y-Pad8) -> Net-(U6-3Y)
- U6 pad 9: GND -> /LEDS_GPIO_3
Routing:
- net +3.3V: track 323.4 -> 429.0 mm, vias 4 -> 7
- net +5V: track 75.7 -> 137.6 mm
- net /LEDS_GPIO_4: track 0.00 -> 46.4 mm, vias 0 -> 1
- net /LEDS_GPIO_1: track 0.00 -> 43.8 mm, vias 0 -> 1
- net /LEDS_GPIO_3: track 0.00 -> 41.9 mm, vias 0 -> 1
- net /LEDS_GPIO: track 38.3 -> 0.00 mm
- net /LEDS_PWR_EN: track 0.00 -> 37.7 mm
- net /LEDS_GPIO_2: track 0.00 -> 36.4 mm, vias 0 -> 1
- net /LEDS_DATA_EN: track 0.00 -> 33.1 mm
- net /LEDS_OUT_4: track 0.00 -> 31.0 mm, vias 0 -> 2
- net /LEDS_OUT_3: track 0.00 -> 27.0 mm, vias 0 -> 2
- net /LEDS_OUT_2: track 0.00 -> 23.1 mm, vias 0 -> 2
- net Net-(U6-3Y): track 0.00 -> 23.0 mm
- net /DCDC_PGood: track 0.00 -> 20.7 mm, vias 0 -> 2
- net /DCDC_EN: track 0.00 -> 17.8 mm, vias 0 -> 2
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